Commit message: Popravljeno ime
še vedno napačni vztrajnostni momenti in momenti osi 123, masa tudu ni ok

File: fanuc_ir_mate_200id_v2/urdf/fanuc_ir_mate_200id_v2.urdf (robot description, URDF)
Before this commit: robot Fanuc - LR Mate-200iD_V1, 7 links, 6 joints
Links:
- link Link 1: mass 14.063 -> 14.0629656801171; geometry collision mesh filename=package://fanuc_ir_mate_200id_v2/meshes/Link 1.STL; visual mesh filename=package://fanuc_ir_mate_200id_v2/meshes/Link 1.STL
- link Link 2: geometry collision mesh filename=package://fanuc_ir_mate_200id_v2/meshes/Link 2.STL; visual mesh filename=package://fanuc_ir_mate_200id_v2/meshes/Link 2.STL
- link Link 3: mass 2.3943 -> 2.39426298307034; geometry collision mesh filename=package://fanuc_ir_mate_200id_v2/meshes/Link 3.STL; visual mesh filename=package://fanuc_ir_mate_200id_v2/meshes/Link 3.STL
- link Link 4: geometry collision mesh filename=package://fanuc_ir_mate_200id_v2/meshes/Link 4.STL; visual mesh filename=package://fanuc_ir_mate_200id_v2/meshes/Link 4.STL
- link Link 5: geometry collision mesh filename=package://fanuc_ir_mate_200id_v2/meshes/Link 5.STL; visual mesh filename=package://fanuc_ir_mate_200id_v2/meshes/Link 5.STL
- link base: geometry collision mesh filename=package://fanuc_ir_mate_200id_v2/meshes/base.STL; visual mesh filename=package://fanuc_ir_mate_200id_v2/meshes/base.STL
- link link 6: geometry collision mesh filename=package://fanuc_ir_mate_200id_v2/meshes/link 6.STL; visual mesh filename=package://fanuc_ir_mate_200id_v2/meshes/link 6.STL
Joints:
- joint Joint 5: origin xyz=0.2454 0 0 rpy=0 0 0 -> xyz=0.245398689130573 0 0 rpy=0 0 0

Commit message: popravljeni

File: fanuc_ir_mate_200id_v2/urdf/fanuc_ir_mate_200id_v2.urdf (robot description, URDF)
Before this commit: robot fanuc_ir_mate_200id_v2, 7 links, 6 joints
Links:
- added link tool0
Joints:
- added joint joint_6-tool0: type fixed, parent link 6, child tool0, origin xyz=0 0 0 rpy=0 0 0
- joint Joint 2: limit lower=-2.5307 upper=1.7453 effort=20 velocity=8 -> lower=-1.77 upper=2.5 effort=20 velocity=8
- joint Joint 3: limit lower=-1.2217 upper=3.5779 effort=15 velocity=9.7 -> lower=-3.5296 upper=1.27 effort=15 velocity=9.7
